Commit message: Update camera.xacro

File: p3dx_description/urdf/p3dx/camera.xacro (robot description, xacro)
@@ -34,4 +34,5 @@
     <!-- Gazebo camera plugin -->
 <gazebo reference="camera_link">
+  <material value="Gazebo/Green"/>
     <sensor type="camera" name="camera">
         <update_rate>30.0</update_rate>
