Commit message: Update pioneer3dx_sonar.xacro

File: p3dx_description/urdf/p3dx/pioneer3dx_sonar.xacro (robot description, xacro)
@@ -2,4 +2,10 @@
 <robot xmlns:xacro="http://wiki.ros.org/xacro">
   <xacro:property name="M_PI" value="3.1415926535897931" />
+  <xacro:property name="ray_count" value="10" />
+  <xacro:property name="field_of_view" value="0" />
+  <xacro:property name="min_range" value="0.1" />
+  <xacro:property name="max_range" value="5.0" />
+  <xacro:property name="ros_topic" value="sonar_scan" />
+  <xacro:property name="update_rate" value="10" />
   <xacro:macro name="pioneer_sonar" params="name parent xyz rpy meshes">
     <!-- Front Sonar -->
@@ -7,7 +13,7 @@
       <origin xyz="${xyz}" rpy="${rpy}"/>
       <parent link="${parent}"/>
-      <child link="${name}"/>
+      <child link="${name}_link"/>
     </joint>
-    <link name="${name}">
+    <link name="${name}_link">
       <inertial>
         <mass value="0.0001"/>
@@ -32,6 +38,37 @@
       </collision>
     </link>
-    <gazebo reference="${name}">
-      <material value="Gazebo/Yellow"/>
+    <gazebo reference="${name}_link">
+      <sensor type="ray" name="${name}">
+        <always_on>true</always_on>
+        <update_rate>${update_rate}</update_rate>
+        <pose>0 0 0 0 0 0</pose>
+        <visualize>true</visualize>
+        <ray>
+          <scan>
+            <horizontal>
+              <samples>${ray_count}</samples>
+              <resolution>1</resolution>
+              <min_angle>-${field_of_view/2}</min_angle>
+              <max_angle> ${field_of_view/2}</max_angle>
+            </horizontal>
+            <vertical>
+              <samples>${ray_count}</samples>
+              <resolution>1</resolution>
+              <min_angle>-${field_of_view/2}</min_angle>
+              <max_angle> ${field_of_view/2}</max_angle>
+            </vertical>
+          </scan>
+          <range>
+            <min>${min_range}</min>
+            <max>${max_range}</max>
+            <resolution>0.01</resolution>
+          </range>
+        </ray>
+        <plugin name="gazebo_ros_${name}_controller" filename="libhector_gazebo_ros_sonar.so">
+          <gaussianNoise>0.005</gaussianNoise>
+          <topicName>${ros_topic}</topicName>
+          <frameId>${name}_link</frameId>
+        </plugin>
+      </sensor>
     </gazebo>
   </xacro:macro>

Commit message: Update pioneer3dx_sonar.xacro

File: p3dx_description/urdf/p3dx/pioneer3dx_sonar.xacro (robot description, xacro)
@@ -3,5 +3,5 @@
   <xacro:property name="M_PI" value="3.1415926535897931" />
   <xacro:property name="ray_count" value="10" />
-  <xacro:property name="field_of_view" value="0" />
+  <xacro:property name="field_of_view" value="1.57" />
   <xacro:property name="min_range" value="0.1" />
   <xacro:property name="max_range" value="5.0" />
@@ -55,5 +55,5 @@
               <samples>${ray_count}</samples>
               <resolution>1</resolution>
-              <min_angle>-${field_of_view/2}</min_angle>
+              <min_angle>-${field_of_view/20}</min_angle>
               <max_angle> ${field_of_view/2}</max_angle>
             </vertical>
